Commit message: update integration code (basic teleop & go to goal)

File: carbi/src/carbi_visualization/description/robot.urdf.xacro (robot description, xacro)
@@ -4,4 +4,9 @@
     <!-- <xacro:property name="width" value="0.2 2.0 0.1" /> -->
     <link name="${fixed_frame}"/>
+    <!-- <joint name = "base_footprint_joint" type = "fixed">
+        <parent link = "base_link"/>
+        <child link = "base_footprint"/>
+        <origin xyz = "0 0 0" rpy = "0 0 0"/>
+    </joint> -->
     <link name="base_link">
         <collision>
@@ -105,3 +110,32 @@
         <axis xyz="0 1 0" />
     </joint>
+    <joint name="laser_joint" type="fixed">
+        <parent link="base_link"/>
+        <child link="laser_frame"/>
+        <origin xyz="0.0 0 0.175" rpy="0 0 0"/>
+    </joint>
+    <link name="laser_frame">
+        <visual>
+            <geometry>
+                <cylinder radius="0.05" length="0.04"/>
+            </geometry>
+            <material name="red"/>
+        </visual>
+        <collision>
+            <geometry>
+                <cylinder radius="0.05" length="0.04"/>
+            </geometry>
+        </collision>
+        <!-- <xacro:inertial_cylinder mass="0.1" length="0.04" radius="0.05">
+            <origin xyz="0 0 0" rpy="0 0 0"/>
+        </xacro:inertial_cylinder> -->
+    </link>
+    <material name="red">
+        <color rgba="1 0 0 1"/>
+    </material>
+    <!-- <launch>
+        <node pkg="laser_filters" type="scan_to_scan_filter_chain" name="laser_filter">
+          <rosparam command="load" file="laserscan_filter.yaml" />
+        </node>
+    </launch> -->
 </robot>
